File: athene-pcb-f072.kicad_pcb (KiCad board)
At the start: 2 copper layers, 303.2 x 92.1 mm, 191 parts, among them J1 HRO-TYPE-C-31-M-12, J2 I2C, J3 ISP, K1 KEYSW, K10 KEYSW, K11 KEYSW, K12 KEYSW, K13 KEYSW, K14 KEYSW, K15 KEYSW, K16 KEYSW, K17 KEYSW, K18 KEYSW, K19 KEYSW, K2 KEYSW, K20 KEYSW, K21 KEYSW, K22 KEYSW, K23 KEYSW, K24 KEYSW, K25 KEYSW, K26 KEYSW, K27 KEYSW, K28 KEYSW, K29 KEYSW, K3 KEYSW, K30 KEYSW, K31 KEYSW, K32 KEYSW, K33 KEYSW, K34 KEYSW, K35 KEYSW, K36 KEYSW, K37 KEYSW, K38 KEYSW, K39 KEYSW, K4 KEYSW, K40 KEYSW, K41 KEYSW, K42 KEYSW, K43 KEYSW, K44 KEYSW, K45 KEYSW, K46 KEYSW, K47 KEYSW, K48 KEYSW, K49 KEYSW, K5 KEYSW, K50 KEYSW, K51 KEYSW, K52 KEYSW, K53 KEYSW, K54 KEYSW, K55 KEYSW, K56 KEYSW, K57 KEYSW, K58 KEYSW, K59 KEYSW, K6 KEYSW, K60 KEYSW, K61 KEYSW, K62 KEYSW, K63 KEYSW, K64 KEYSW, K65 KEYSW, K66 KEYSW, K67 KEYSW, K7 KEYSW, K8 KEYSW, K9 KEYSW, Q1 DTC123J, U1 STM32F072CBU6, U2 SRV05-4-P-T7, U3 XC6206P332MR, U4 SN74LVC1G07DBVR

Commit message: v1.0a update
Parts:
- removed U4: SN74LVC1G07DBVR, Package_TO_SOT_SMD:SOT-23-5
- added J4: RGB Extension Pads, Connector_Wire:SolderWirePad_1x03_P3.175mm_Drill0.8mm, B.Cu at (304.8, 105.6)
- added R8: 5.1k, Resistor_SMD:R_0805_2012Metric, B.Cu at (57.4, 106.5)
- C11, C12, C13, C14, C15, C16, C17, C3, C4, C6: value 0.1uF -> 100nF
Connections:
- RGB1 pad 2: Net-(RGB1-Pad2) -> RGB
- RGB7 pad 4: Net-(RGB7-Pad4) -> RGB_EX
- U2 pad 1: D+ -> Net-(U2-Pad1)
- U2 pad 6: D- -> Net-(U2-Pad6)
Routing:
- net RGB_EX: track 0.00 -> 26.0 mm
- net GND: track 66.8 -> 88.9 mm, vias 9 -> 10
- net +5V: track 349.1 -> 364.8 mm
- net RGB: track 100.4 -> 107.9 mm, vias 4 -> 6
- net Net-(RGB1-Pad2): track 3.88 -> 0.00 mm
- net D+: track 41.6 -> 38.4 mm
- net +3V3: track 143.1 -> 145.3 mm
- net ROW2: track 309.7 -> 311.4 mm
- net ROW4: track 361.9 -> 363.1 mm
- net ROW3: track 325.8 -> 327.0 mm
- net D-: track 42.1 -> 41.2 mm
- net SWDIO: track 38.9 -> 38.2 mm
- net SWCLK: track 47.6 -> 47.1 mm

Commit message: File cleanup
Parts:
- removed the D68 at (51.9, 82.2)
- added J5: EX, Project Library:6-Pin Header, F.Cu at (58.1, 83.2)
- added R6: 100k, Resistor_SMD:R_0805_2012Metric, B.Cu at (62.6, 72.9)
- C18: value 4.7nF -> 4.7uF
- C19: value 100uF -> 1uF
- J3: footprint keebio-parts:ICSP-Header -> Project Library:ICSP-Header
- Q1: value DTC123J -> 2N7002
- R4: value 100k -> 10k
- R5: renamed from R7; value 33k -> 10k
- moved C18 20.1 mm to (62.6, 70.8), turned to 0 degrees
- moved R4 14.1 mm to (62.6, 68.8), turned to 0 degrees
- moved Q1 11.2 mm to (58.4, 76.4), turned to -90 degrees
- moved R5 5.77 mm to (53.6, 76.4)
- moved C19 5.74 mm to (55.6, 76.5), turned to 90 degrees
- moved S1 4.03 mm to (56.5, 71.0), turned to 0 degrees
- renumbered D69 to D68, R5 to R7, R6 to R8, R8 to R9
Connections:
- C18 pad 1: NRST -> BOOT0
- C18 pad 2: GND -> Net-(C18-Pad2)
- C19 pad 1: BOOT0 -> NRST
- Q1 pad 1: Net-(D68-Pad2) -> Net-(C18-Pad2)
- R5 pad 1: Net-(D68-Pad1) -> +3V3
- R5 pad 2: BOOT0 -> NRST
- S1 pad 1: +3V3 -> BOOT0
- S1 pad 2: Net-(D68-Pad2) -> +3V3
- U1 pad 14: Net-(U1-Pad14) -> EX1
- U1 pad 15: Net-(U1-Pad15) -> EX2
- U1 pad 16: Net-(U1-Pad16) -> EX3
- U1 pad 17: Net-(U1-Pad17) -> EX4
- U1 pad 18: Net-(U1-Pad18) -> EX5
- U1 pad 19: Net-(U1-Pad19) -> EX6
Routing:
- net EX1: track 0.00 -> 37.4 mm, vias 0 -> 1
- net EX2: track 0.00 -> 35.9 mm, vias 0 -> 1
- net EX3: track 0.00 -> 34.5 mm, vias 0 -> 1
- net EX4: track 0.00 -> 33.1 mm, vias 0 -> 1
- net EX5: track 0.00 -> 31.6 mm, vias 0 -> 1
- net EX6: track 0.00 -> 31.1 mm, vias 0 -> 1
- net BOOT0: track 76.6 -> 65.5 mm, vias 3 -> 2
- net Net-(D68-Pad2): track 9.50 -> 0.00 mm
- net Net-(C18-Pad2): track 0.00 -> 8.11 mm
- net GND: track 88.9 -> 93.4 mm
- net +3V3: track 145.3 -> 149.7 mm
- net Net-(D68-Pad1): track 2.50 -> 0.00 mm
- net NRST: track 60.5 -> 58.5 mm
- net ROW3: track 327.0 -> 325.9 mm
- net ROW4: track 363.1 -> 361.9 mm
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