File: athene-pcb-f072.kicad_sch (KiCad schematic)
At the start: 185 parts, among them J1 HRO-TYPE-C-31-M-12, J2 I2C, J3 ISP, K1 KEYSW, K10 KEYSW, K11 KEYSW, K12 KEYSW, K13 KEYSW, K14 KEYSW, K15 KEYSW, K16 KEYSW, K17 KEYSW, K18 KEYSW, K19 KEYSW, K2 KEYSW, K20 KEYSW, K21 KEYSW, K22 KEYSW, K23 KEYSW, K24 KEYSW, K25 KEYSW, K26 KEYSW, K27 KEYSW, K28 KEYSW, K29 KEYSW, K3 KEYSW, K30 KEYSW, K31 KEYSW, K32 KEYSW, K33 KEYSW, K34 KEYSW, K35 KEYSW, K36 KEYSW, K37 KEYSW, K38 KEYSW, K39 KEYSW, K4 KEYSW, K40 KEYSW, K41 KEYSW, K42 KEYSW, K43 KEYSW, K44 KEYSW, K45 KEYSW, K46 KEYSW, K47 KEYSW, K48 KEYSW, K49 KEYSW, K5 KEYSW, K50 KEYSW, K51 KEYSW, K52 KEYSW, K53 KEYSW, K54 KEYSW, K55 KEYSW, K56 KEYSW, K57 KEYSW, K58 KEYSW, K59 KEYSW, K6 KEYSW, K60 KEYSW, K61 KEYSW, K62 KEYSW, K63 KEYSW, K64 KEYSW, K65 KEYSW, K66 KEYSW, K67 KEYSW, K7 KEYSW, K8 KEYSW, K9 KEYSW, Q1 DTC123J, U1 STM32F072CBU6, U2 SRV05-4-P-T7, U3 XC6206P332MR, U4 SN74LVC1G07DBVR

Commit message: v1.0a update
Parts:
- added J4: RGB Extension Pads, Connector_Wire:SolderWirePad_1x03_P3.175mm_Drill0.8mm, symbol Connector:Conn_01x03_Male
- added R8: 5.1k, Resistor_SMD:R_0805_2012Metric, symbol Device:R_Small
- C11, C12, C13, C14, C15, C16, C17, C3, C4, C6: value 0.1uF -> 100nF
- H1, H2, H3, H4, H5, H6, J1, J2, J3, RGB1, RGB2, RGB3, RGB4, RGB5, RGB6, RGB7, U4: now left out of the parts list
Connections:
- net +5V: now also J4.3 (Pin_3), R8.2
- net D+: no longer U2.1 (IO1)
- net D-: no longer U2.6 (IO4)
- net GND: now also J4.1 (Pin_1)
- net RGB: now also RGB1.2 (DIN), R8.1; no longer U4.2
- net at U4.4: no longer RGB1.2 (DIN)
- net RGB_EX: now reaches RGB7.4 (DOUT)
- net RGB_EX: now also J4.2 (Pin_2)
- no-connect marks 3 -> 8
Other:
- company: (none) -> @kebn#2121
- moved on the sheet: R1, R2, R3, R5, R6, U2

Commit message: File cleanup
Parts:
- removed D68: 1N4148W, Diode_SMD:D_SOD-123, symbol Device:D_Small
- removed Q1: DTC123J, Package_TO_SOT_SMD:SOT-23, symbol Transistor_BJT:DTC123J
- removed R7: 33k, Resistor_SMD:R_0805_2012Metric, symbol Device:R_Small
- removed U4: SN74LVC1G07DBVR, Package_TO_SOT_SMD:SOT-23-5, symbol 74xGxx:74LVC1G07
- added J5: EX, Project Library:6-Pin Header, symbol Connector_Generic:Conn_01x06
- added Q1: 2N7002, Package_TO_SOT_SMD:SOT-23, symbol Transistor_FET:2N7002
- added R4, R5: 10k, Resistor_SMD:R_0805_2012Metric, symbol Device:R_Small
- C18: value 4.7nF -> 4.7uF
- C19: value 100uF -> 1uF
- J3: footprint keebio-parts:ICSP-Header -> Project Library:ICSP-Header
- renumbered D69 to D68, R4 to R6, R5 to R7, R6 to R8, R8 to R9
Connections:
- net +3V3: now also S1.2, R5.1; no longer S1.1
- net BOOT0: now also C18.1, S1.1, R4.1; no longer C19.1, R6.1
- net GND: now also Q1.2 (S), R4.2; no longer C18.2
- net NRST: now also C19.1, Q1.3 (D), R5.2; no longer C18.1
- net EX1: now reaches U1.14 (PA4)
- net EX1: now also J5.1 (Pin_1)
- net EX2: now reaches U1.15 (PA5)
- net EX2: now also J5.2 (Pin_2)
- net EX3: now reaches U1.16 (PA6)
- net EX3: now also J5.3 (Pin_3)
- net EX4: now reaches U1.17 (PA7)
- net EX4: now also J5.4 (Pin_4)
- net EX5: now reaches U1.18 (PB0)
- net EX5: now also J5.5 (Pin_5)
- net EX6: now reaches U1.19 (PB1)
- net EX6: now also J5.6 (Pin_6)
- new net: C18.2, Q1.1 (G), R6.1
- no-connect marks 8 -> 4
Other:
- note added: "EXTRA PINS"
- moved on the sheet: C18, C19, H1, H2, H3, H4, H5, H6, J3, K16, R6, R7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
